File: mainboardv3.4.sch (EAGLE design)
At the start: 128 parts, among them IC1 LM2596S, IC2 TDA2822D, IC3 MCP2562P, IC4 STM32F103RBT6, IC5 MIC2288YD5, IC6 ULN2003AD, IC7 LM2901, IC8 REG1117, IC9 NC7SZ10P6X, Q1 8MHz

Commit message: New mainboard v3.4 Using TagConnect for programming Using FET for dcsw output Optimized BOM Added solder bridges for optional resistors
Parts:
- removed C18: 1nF, rcl:C-EUC0603
- removed JP6: 1365-10, con-leotronics:1365-10
- removed R28: 510, rcl:R-EU_R0603
- removed R30, R34: 10k, rcl:R-EU_R0603
- added J1: (no value), tag-connect:TC2030_SWD-MCP
- added SJ2, SJ3: SOLDERJUMPERNO, SparkFun-Passives:SOLDERJUMPERNO
- added SJ4: SOLDERJUMPERTRACE, SparkFun-Passives:SOLDERJUMPERTRACE
- added T1: AP9T18GH-HF, transistor-power:AP9T18GH-HF
- added U$1: OI-LOGO, SparkFun-Aesthetics:OI-LOGO
- IC3: value MCP2562P -> SN65HVD230DR
- Q1: device crystal:CRYSTALHC49UP -> SparkFun-FreqCtrl:CRYSTALTXC-7A
- R11: value 120R/510R -> 510R
Connections:
- new net N$3: R17.2, SJ3.2
- new net N$5: IC4PORTA_H.PA13, J1.SWDIO/TMS
- new net N$8: R18.2, SJ2.2
- net ENC_A/S2: now also SJ2.1; no longer R18.2
- net ENC_B/S3: now also SJ3.1; no longer R17.2
- net ENC_Z/R1: no longer R28.2, R30.2
- net GND: now also IC6.I7, J1.GND, T1.S; no longer C18.2, JP6-3.S, JP6-5.S
- net N$6: now also IC4PORTA_H.PA14, J1.SWCLK/TCK; no longer IC4PORTA_H.PA13, JP6-2.S
- net N$9: now also C1.1, R1.2, SJ4.2; no longer IC4PORTA_H.PA14, JP6-4.S
- net NRST: no longer JP6-10.S, R34.1
- net OUT_BRAKE: now also IC6.O6; no longer IC6.O7
- net OUT_DCSW: now also IC6.O7, T1.D; no longer IC6.O5, IC6.O6
- net OUT_ERR: now also IC6.O5; no longer IC6.O4
- net OUT_OVTMP: now also IC6.O4; no longer IC6.O3
- net OUT_PRE: now also IC6.O2
- net OUT_TEMP: now also IC6.O3; no longer IC6.O2
- net PB1/ADC9: now also IC6.I2
- net PB9/TIM4_CH4: now also IC6.I3; no longer IC6.I2
- net PC10: now also IC6.I5; no longer IC6.I4
- net PC11: now also IC6.I4; no longer IC6.I3
- net PC13: now also T1.G; no longer IC6.I5, IC6.I6
- net PC5/ADC15: now also IC6.I6; no longer IC6.I7
- net PD2/TIM3_ETR: no longer C18.1, R30.1
- net S4/S1: now also SJ4.1; no longer C1.1, R1.2
- net VCC: no longer C48.1, IC3.VDD, R28.1
- net VCCIO: now also C48.1, IC3.VDD, J1.VCC; no longer IC3.VREF, JP6-1.S, R34.2
Other:
- note added: "For incremental open collector encoders close SJ2 and SJ3 for pull-up"
- note added: "Open SJ4 to generate supply voltage ON JP2.2. If needed bridge or replace R11 to output full 5V."
- note removed: "In single channel encoder mode omit C18 In resolver mode populate the resolver excitation parts, C1 and R1 and omit R17, R18, R28, R30 and C18."
- note removed: "JP6=20021121-00010C4LF"
- note removed: "Populate C1 and R1 only for resolver mode. It adds 1.6V offset to resolver signal R11=510R in resolver mode"
- moved on the sheet: C12, R17, R18, R21
