File: mainboardv3.4.sch (EAGLE design)
At the start: 129 parts, among them IC1 LM2596S, IC2 TDA2822D, IC3 SN65HVD230DR, IC4 STM32F103RBT6, IC5 MIC2288YD5, IC6 ULN2003AD, IC7 LM2901, IC8 REG1117, IC9 NC7SZ10P6X, Q1 8MHz, T1 AP9T18GH-HF

Commit message: Added new files
Parts:
- C24: value 1µ -> 10µ
- IC9: value NC7SZ10P6X -> 74AHC1G00DCK; device 74xx-eu:741G10X -> 74xx-little-de:74AHC1G00DCK
- L3: value 10µH -> 100µH
Connections:
- net GND: now also IC9P.GND; no longer IC9PWR.GND
- net PA1/TIM2_CH2: now also IC9A.I0; no longer IC9>NAME.I0
- net PA3/ADC3: no longer IC9>NAME.I1
- net PB12/TIM1_BKIN: now also IC9A.O; no longer IC9>NAME.O
- net PC9: now also IC9A.I1; no longer IC9>NAME.I2
- net VCCIO: now also IC9P.VCC; no longer IC9PWR.VCC
Changed lines of the file:
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@@
 <part name="VCC2" library="supply1" deviceset="VCCIO" device=""/>
 <part name="GND15" library="supply1" deviceset="GND" device=""/>
-<part name="C24" library="rcl" deviceset="C-EU" device="C0603" value="1µ"/>
+<part name="C24" library="rcl" deviceset="C-EU" device="C0603" value="10µ"/>
 <part name="R2" library="rcl" deviceset="R-EU_" device="R0603" value="3k3"/>
 <part name="R3" library="rcl" deviceset="R-EU_" device="R0603" value="3k3"/>
@@
 <part name="GND50" library="supply1" deviceset="GND" device=""/>
 <part name="GND58" library="supply1" deviceset="GND" device=""/>
-<part name="L3" library="rcl" deviceset="L-EU" device="L2012C" value="10µH"/>
+<part name="L3" library="rcl" deviceset="L-EU" device="L2012C" value="100µH"/>
 <part name="VCC8" library="supply1" deviceset="VCCIO" device=""/>
 <part name="P+17" library="supply1" deviceset="+12V" device=""/>
@@
 <part name="LOGO1" library="SparkFun-Aesthetics" deviceset="OSHW-LOGO" device="M"/>
 <part name="SJ1" library="SparkFun-Passives" deviceset="SOLDERJUMPER" device="TRACE"/>
-<part name="IC9" library="74xx-eu" deviceset="74*1G10" device="X" value="NC7SZ10P6X"/>
 <part name="J1" library="tag-connect" deviceset="TC2030_SWD" device="-MCP"/>
 <part name="VCC3" library="supply1" deviceset="VCCIO" device=""/>
@@
 <part name="VCC5" library="supply1" deviceset="VCCIO" device=""/>
 <part name="U$1" library="SparkFun-Aesthetics" deviceset="OI-LOGO" device=""/>
+<part name="IC9" library="74xx-little-de" deviceset="74*1G00" device="DCK" technology="AHC"/>
 </parts>
 <sheets>
@@
 <instance part="GND45" gate="1" x="182.88" y="43.18"/>
 <instance part="P+15" gate="VCC" x="-38.1" y="-40.64"/>
-<instance part="GND17" gate="1" x="248.92" y="-17.78"/>
-<instance part="VCC4" gate="G$1" x="248.92" y="7.62" smashed="yes"/>
+<instance part="GND17" gate="1" x="248.92" y="-15.24"/>
+<instance part="VCC4" gate="G$1" x="248.92" y="5.08" smashed="yes"/>
 <instance part="P+9" gate="VCC" x="223.52" y="-7.62" smashed="yes"/>
 <instance part="GND2" gate="1" x="83.82" y="0" rot="MR0"/>
@@
 <instance part="LOGO1" gate="G$1" x="-45.72" y="60.96"/>
 <instance part="SJ1" gate="1" x="-81.28" y="106.68"/>
-<instance part="IC9" gate="&gt;NAME" x="246.38" y="-5.08" smashed="yes">
-<attribute name="VALUE" x="241.3" y="-25.4" size="1.778" layer="96" rot="R90"/>
-</instance>
-<instance part="IC9" gate="PWR" x="248.92" y="-5.08" smashed="yes"/>
 <instance part="J1" gate="G$1" x="5.08" y="68.58" rot="R90"/>
 <instance part="VCC3" gate="G$1" x="-10.16" y="60.96"/>
@@
 <instance part="VCC5" gate="G$1" x="213.36" y="-81.28" smashed="yes" rot="MR0"/>
 <instance part="U$1" gate="G$1" x="-35.56" y="68.58"/>
+<instance part="IC9" gate="A" x="246.38" y="-5.08"/>
+<instance part="IC9" gate="P" x="248.92" y="-5.08"/>
 </instances>
 <busses>
@@
 <wire x1="254" y1="-5.08" x2="259.08" y2="-5.08" width="0.1524" layer="91"/>
 <label x="259.08" y="-5.08" size="1.778" layer="95" rot="R90"/>
-<pinref part="IC9" gate="&gt;NAME" pin="O"/>
+<pinref part="IC9" gate="A" pin="O"/>
 </segment>
 </net>
@@
 <wire x1="223.52" y1="-22.86" x2="223.52" y2="-27.94" width="0.1524" layer="91"/>
 <label x="215.9" y="-25.4" size="1.778" layer="95" rot="R180"/>
-<wire x1="238.76" y1="-7.62" x2="233.68" y2="-7.62" width="0.1524" layer="91"/>
+<wire x1="241.3" y1="-7.62" x2="233.68" y2="-7.62" width="0.1524" layer="91"/>
 <wire x1="233.68" y1="-7.62" x2="233.68" y2="-27.94" width="0.1524" layer="91"/>
 <wire x1="233.68" y1="-27.94" x2="223.52" y2="-27.94" width="0.1524" layer="91"/>
 <junction x="223.52" y="-27.94"/>
 <wire x1="223.52" y1="-27.94" x2="213.36" y2="-27.94" width="0.1524" layer="91"/>
-<pinref part="IC9" gate="&gt;NAME" pin="I2"/>
+<pinref part="IC9" gate="A" pin="I1"/>
 </segment>
 <segment>
@@
 </segment>
 <segment>
-<pinref part="GND17" gate="1" pin="GND"/>
-<pinref part="IC9" gate="PWR" pin="GND"/>
-</segment>
-<segment>
 <pinref part="J1" gate="G$1" pin="GND"/>
 <pinref part="GND5" gate="1" pin="GND"/>
@@
 <wire x1="-111.76" y1="109.22" x2="-111.76" y2="106.68" width="0.1524" layer="91"/>
 <junction x="-111.76" y="106.68"/>
+</segment>
+<segment>
+<pinref part="IC9" gate="P" pin="GND"/>
+<pinref part="GND17" gate="1" pin="GND"/>
 </segment>
 </net>
@@
 <wire x1="203.2" y1="0" x2="203.2" y2="22.86" width="0.1524" layer="91"/>
 <wire x1="215.9" y1="0" x2="215.9" y2="-2.54" width="0.1524" layer="91"/>
-<wire x1="215.9" y1="-2.54" x2="238.76" y2="-2.54" width="0.1524" layer="91"/>
+<wire x1="215.9" y1="-2.54" x2="241.3" y2="-2.54" width="0.1524" layer="91"/>
 <wire x1="193.04" y1="0" x2="203.2" y2="0" width="0.1524" layer="91"/>
 <junction x="203.2" y="0"/>
 <wire x1="215.9" y1="-2.54" x2="203.2" y2="-2.54" width="0.1524" layer="91"/>
 <junction x="215.9" y="-2.54"/>
-<pinref part="IC9" gate="&gt;NAME" pin="I0"/>
+<pinref part="IC9" gate="A" pin="I0"/>
 </segment>
 </net>
@@
 <wire x1="-67.31" y1="-15.24" x2="-73.66" y2="-15.24" width="0.1524" layer="91"/>
 <junction x="-73.66" y="-15.24"/>
-</segment>
-<segment>
-<wire x1="238.76" y1="-5.08" x2="233.68" y2="-5.08" width="0.1524" layer="91"/>
-<label x="220.98" y="-5.08" size="1.778" layer="95"/>
-<pinref part="IC9" gate="&gt;NAME" pin="I1"/>
 </segment>
 </net>
@@
 </segment>
 <segment>
-<pinref part="VCC4" gate="G$1" pin="VCCIO"/>
-<pinref part="IC9" gate="PWR" pin="VCC"/>
-</segment>
-<segment>
 <pinref part="J1" gate="G$1" pin="VCC"/>
 <wire x1="-2.54" y1="55.88" x2="-2.54" y2="53.34" width="0.1524" layer="91"/>
@@
 <pinref part="VCC5" gate="G$1" pin="VCCIO"/>
 </segment>
-</net>
+<segment>
+<pinref part="IC9" gate="P" pin="VCC"/>
+<pinref part="VCC4" gate="G$1" pin="VCCIO"/>
+</segment>
+</net>
