File: mainboard-mini.sch (EAGLE design)
At the start: 104 parts, among them IC1 XC6206P332MR, IC2 LM2901, IC3 NC7SZ10P6X, IC4 STM32F103RBT6, IC5 TDA2822D, IC6 SN65HVD230, IC7 RT8259GE, Q1 8MHz

Commit message: Added new files
Parts:
- IC1: device linear:MCP1703CB -> burr-brown:REG1117
Connections:
- net VCC: now also IC1.VIN; no longer IC1.VI
- net VCCIO: now also IC1.VOUT; no longer IC1.VO
Other:
- moved on the sheet: IC1
Changed lines of the file:
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@@
 <part name="RN6" library="resistor-net" deviceset="CTS742C083" device="" value="1k2"/>
 <part name="RN4" library="resistor-net" deviceset="CTS742C083" device="" value="1k2"/>
-<part name="IC1" library="linear" deviceset="MCP1703" device="CB" value="XC6206P332MR"/>
+<part name="IC1" library="burr-brown" deviceset="REG1117" device="" value="XC6206P332MR"/>
 <part name="RN2" library="resistor-net" deviceset="CTS742C083" device="" value="470"/>
 <part name="RN1" library="resistor-net" deviceset="CTS742C083" device="" value="470"/>
@@
 <wire x1="109.22" y1="104.14" x2="109.22" y2="111.76" width="0.1524" layer="91"/>
 <wire x1="121.92" y1="104.14" x2="109.22" y2="104.14" width="0.1524" layer="91"/>
+<junction x="109.22" y="104.14"/>
 <wire x1="109.22" y1="104.14" x2="93.98" y2="104.14" width="0.1524" layer="91"/>
-<junction x="109.22" y="104.14"/>
-<wire x1="93.98" y1="104.14" x2="78.74" y2="104.14" width="0.1524" layer="91"/>
-<junction x="93.98" y="104.14"/>
 <junction x="78.74" y="104.14"/>
 <pinref part="R5" gate="G$1" pin="1"/>
 <junction x="43.18" y="104.14"/>
+<pinref part="C2" gate="G$1" pin="2"/>
 <pinref part="IC1" gate="G$1" pin="GND"/>
-<wire x1="93.98" y1="111.76" x2="93.98" y2="104.14" width="0.1524" layer="91"/>
-<pinref part="C2" gate="G$1" pin="2"/>
+<wire x1="93.98" y1="104.14" x2="78.74" y2="104.14" width="0.1524" layer="91"/>
+<wire x1="93.98" y1="106.68" x2="93.98" y2="104.14" width="0.1524" layer="91"/>
+<junction x="93.98" y="104.14"/>
 </segment>
 <segment>
@@
 <wire x1="66.04" y1="114.3" x2="71.12" y2="114.3" width="0.1524" layer="91"/>
 <junction x="71.12" y="114.3"/>
-<pinref part="IC1" gate="G$1" pin="VI"/>
-<wire x1="83.82" y1="119.38" x2="78.74" y2="119.38" width="0.1524" layer="91"/>
+<pinref part="IC1" gate="G$1" pin="VIN"/>
+<wire x1="81.28" y1="119.38" x2="78.74" y2="119.38" width="0.1524" layer="91"/>
 </segment>
 <segment>
@@
 <pinref part="C4" gate="G$1" pin="1"/>
 <wire x1="109.22" y1="124.46" x2="109.22" y2="119.38" width="0.1524" layer="91"/>
-<junction x="109.22" y="119.38"/>
 <wire x1="111.76" y1="124.46" x2="109.22" y2="124.46" width="0.1524" layer="91"/>
 <junction x="109.22" y="124.46"/>
-<pinref part="IC1" gate="G$1" pin="VO"/>
-<wire x1="104.14" y1="119.38" x2="109.22" y2="119.38" width="0.1524" layer="91"/>
-</segment>
-<segment>
+<pinref part="IC1" gate="G$1" pin="VOUT"/>
+<wire x1="106.68" y1="119.38" x2="109.22" y2="119.38" width="0.1524" layer="91"/>
+<junction x="109.22" y="119.38"/>
+</segment>
+<segment>
