File: mainboardv3.4.brd (EAGLE design)
At the start: 79.7 x 80 mm, 129 parts, among them IC1 LM2596S, IC2 TDA2822D, IC3 SN65HVD230DR, IC4 STM32F103RBT6, IC5 MIC2288YD5, IC6 ULN2003AD, IC7 LM2901, IC8 REG1117, IC9 NC7SZ10P6X, Q1 8MHz, T1 AP9T18GH-HF

Commit message: Added new files
Parts:
- C24: value 1µ -> 10µ
- IC9: value NC7SZ10P6X -> 74AHC1G00DCK; device 74xx-eu:SC70-6 -> 74xx-little-de:SC70-5
- L3: value 10µH -> 100µH
- moved IC9 0.62 mm to (55.3, 25.3)
Connections:
- net GND: now also IC9.3; no longer IC9.2
- net PA3/ADC3: no longer IC9.3
- net PC9: now also IC9.2; no longer IC9.6
Routing:
- net PA3/ADC3: track 53.5 -> 49.3 mm
- net PC9: track 51.9 -> 54.5 mm
- net VCCIO: track 97.4 -> 96.6 mm
- net PA1/TIM2_CH2: track 107.5 -> 108.2 mm
Changed lines of the file:
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@@
 <element name="C29" library="rcl" package="C0603" value="1µ" x="41.275" y="31.115"/>
 <element name="C30" library="rcl" package="C0603" value="1µ" x="54.61" y="31.75" rot="R180"/>
-<element name="C24" library="rcl" package="C0603" value="1µ" x="56.52" y="45.5" smashed="yes" rot="R180">
+<element name="C24" library="rcl" package="C0603" value="10µ" x="56.52" y="45.5" smashed="yes" rot="R180">
 <attribute name="NAME" x="59.695" y="47.405" size="1.27" layer="25" rot="R180"/>
 <attribute name="VALUE" x="57.155" y="47.405" size="1.27" layer="27" rot="R180"/>
@@
 <element name="R52" library="rcl" package="R0603" value="10R" x="26.7375" y="13.045" rot="R270"/>
 <element name="C44" library="rcl" package="C0603" value="22n" x="29.21" y="16.5" rot="R270"/>
-<element name="L3" library="rcl" package="L2012C" value="10µH" x="55.9575" y="49.06" smashed="yes" rot="R90">
+<element name="L3" library="rcl" package="L2012C" value="100µH" x="55.9575" y="49.06" smashed="yes" rot="R90">
 <attribute name="NAME" x="58.2275" y="50.695" size="1.27" layer="25" rot="R90"/>
 <attribute name="VALUE" x="58.4975" y="47.155" size="1.27" layer="27" rot="R90"/>
@@
 <element name="LOGO1" library="SparkFun-Aesthetics" package="OSHW-LOGO-M" value="OSHW-LOGOM" x="34.375" y="75.3125"/>
 <element name="SJ1" library="SparkFun-Passives" package="SJ_2S-TRACE" value="SOLDERJUMPERTRACE" x="3.4375" y="45.3125" rot="R90"/>
-<element name="IC9" library="74xx-eu" package="SC70-6" value="NC7SZ10P6X" x="55.9375" y="25.3125" smashed="yes" rot="R180">
-<attribute name="NAME" x="56.8265" y="23.7885" size="0.8128" layer="25" rot="R180"/>
-<attribute name="VALUE" x="56.6995" y="25.5665" size="0.4064" layer="27" rot="R180"/>
-</element>
 <element name="J1" library="tag-connect" package="TC2030-MCP" value="" x="70" y="31.5625" rot="R90"/>
 <element name="SJ2" library="SparkFun-Passives" package="SJ_2S-NO" value="SOLDERJUMPERNO" x="19.0625" y="22.8125"/>
@@
 <element name="IC6" library="uln-udn" package="SO16" value="ULN2003AD" x="6.875" y="38.75" rot="R270"/>
 <element name="U$1" library="SparkFun-Aesthetics" package="OI_LOGO" value="OI-LOGO" x="59.0625" y="15"/>
+<element name="IC9" library="74xx-little-de" package="SC70-5" value="74AHC1G00DCK" x="55.3125" y="25.3125" rot="R180"/>
 </elements>
 <signals>
@@
 <contactref element="C39" pad="1"/>
 <contactref element="C48" pad="2"/>
-<contactref element="IC9" pad="2"/>
-<contactref element="IC9" pad="2"/>
 <contactref element="J1" pad="5"/>
 <wire x1="70.635" y1="35.3725" x2="70.8875" y2="35.625" width="0.3048" layer="1"/>
@@
 <contactref element="IC6" pad="8"/>
 <contactref element="IC6" pad="7"/>
+<contactref element="IC9" pad="3"/>
+<contactref element="IC9" pad="3"/>
 </signal>
 <signal name="VCC">
@@
 <wire x1="47.3875" y1="19.9825" x2="48.3075" y2="19.0625" width="0.3048" layer="1"/>
 <wire x1="48.3075" y1="19.0625" x2="53.125" y2="19.0625" width="0.3048" layer="1"/>
-<wire x1="53.125" y1="19.0625" x2="55.2875" y2="21.225" width="0.3048" layer="1"/>
 <contactref element="IC9" pad="4"/>
-<wire x1="55.2875" y1="21.225" x2="55.2875" y2="24.3875" width="0.3048" layer="1"/>
+<wire x1="53.125" y1="19.0625" x2="54.6625" y2="20.6" width="0.3048" layer="1"/>
+<wire x1="54.6625" y1="20.6" x2="54.6625" y2="24.4625" width="0.3048" layer="1"/>
 </signal>
 <signal name="TIM1_CH1N">
@@
 <wire x1="45.72" y1="8.89" x2="45.72" y2="10.16" width="0.3048" layer="16"/>
 <wire x1="48.18" y1="28.38" x2="52.505" y2="24.055" width="0.3048" layer="1"/>
-<wire x1="52.505" y1="24.055" x2="52.505" y2="20.46" width="0.3048" layer="1"/>
+<wire x1="52.505" y1="24.055" x2="52.505" y2="23.75" width="0.3048" layer="1"/>
+<wire x1="52.505" y1="23.75" x2="52.505" y2="20.46" width="0.3048" layer="1"/>
 <wire x1="45.72" y1="10.16" x2="52.505" y2="16.945" width="0.3048" layer="16"/>
 <wire x1="52.505" y1="16.945" x2="52.505" y2="17.8125" width="0.3048" layer="16"/>
@@
 <wire x1="51.2775" y1="20.28" x2="51.4575" y2="20.46" width="0.4064" layer="1"/>
 <wire x1="51.4575" y1="20.46" x2="52.505" y2="20.46" width="0.4064" layer="1"/>
-<contactref element="IC9" pad="6"/>
-<wire x1="56.5875" y1="22.8375" x2="56.5875" y2="24.3875" width="0.3048" layer="1"/>
 <wire x1="56.25" y1="20.3125" x2="56.25" y2="22.5" width="0.3048" layer="1"/>
 <wire x1="56.25" y1="22.5" x2="56.5875" y2="22.8375" width="0.3048" layer="1"/>
+<contactref element="IC9" pad="2"/>
+<wire x1="55.3125" y1="26.1625" x2="55.3125" y2="25.625" width="0.3048" layer="1"/>
+<wire x1="55.3125" y1="25.625" x2="55" y2="25.3125" width="0.3048" layer="1"/>
+<wire x1="55" y1="25.3125" x2="54.375" y2="25.3125" width="0.3048" layer="1"/>
+<wire x1="54.375" y1="25.3125" x2="52.8125" y2="23.75" width="0.3048" layer="1"/>
+<wire x1="52.8125" y1="23.75" x2="52.505" y2="23.75" width="0.3048" layer="1"/>
 </signal>
 <signal name="PC10">
@@
 <wire x1="61.08" y1="60.48" x2="69.74" y2="60.48" width="0.3048" layer="1"/>
 <wire x1="53.76" y1="53.16" x2="61.08" y2="60.48" width="0.3048" layer="1"/>
-<contactref element="IC9" pad="1"/>
 <wire x1="59.73" y1="23.43" x2="56.9225" y2="26.2375" width="0.3048" layer="1"/>
-<wire x1="56.9225" y1="26.2375" x2="56.5875" y2="26.2375" width="0.3048" layer="1"/>
 <wire x1="77.12" y1="51.84" x2="77.1875" y2="51.7725" width="0.3048" layer="1"/>
 <wire x1="77.1875" y1="51.7725" x2="77.1875" y2="30.3125" width="0.3048" layer="1"/>
@@
 <wire x1="62.8125" y1="25" x2="61.2425" y2="23.43" width="0.3048" layer="1"/>
 <wire x1="61.2425" y1="23.43" x2="59.73" y2="23.43" width="0.3048" layer="1"/>
+<contactref element="IC9" pad="1"/>
+<wire x1="56.9225" y1="26.2375" x2="55.9625" y2="26.2375" width="0.3048" layer="1"/>
+<wire x1="55.9625" y1="26.2375" x2="55.9625" y2="26.1625" width="0.3048" layer="1"/>
 </signal>
 <signal name="UDC">
@@
 <wire x1="51.435" y1="29.21" x2="51.7351" y2="29.21" width="0.3048" layer="1"/>
 <wire x1="51.7651" y1="29.21" x2="51.435" y2="29.21" width="0.3048" layer="1"/>
-<contactref element="IC9" pad="3"/>
-<wire x1="55.2875" y1="26.2375" x2="52.315" y2="29.21" width="0.3048" layer="1"/>
 <wire x1="52.315" y1="29.21" x2="51.435" y2="29.21" width="0.3048" layer="1"/>
 </signal>
@@
 <wire x1="55.9575" y1="50.06" x2="55.875" y2="50.06" width="0.3048" layer="1"/>
 <wire x1="55.875" y1="50.06" x2="55.875" y2="52.5" width="0.4064" layer="1"/>
-<contactref element="IC9" pad="5"/>
-<wire x1="55.9375" y1="24.3875" x2="55.9375" y2="24.6875" width="0.3048" layer="1"/>
-<wire x1="55.9375" y1="24.6875" x2="55.625" y2="25" width="0.3048" layer="1"/>
-<wire x1="55.625" y1="25" x2="54.375" y2="25" width="0.3048" layer="1"/>
-<via x="54.375" y="25" extent="1-16" drill="0.6" shape="octagon"/>
-<wire x1="54.375" y1="25" x2="54.375" y2="25.3125" width="0.3048" layer="16"/>
 <contactref element="J1" pad="1"/>
 <wire x1="70.635" y1="32.8325" x2="70.9375" y2="32.53" width="0.3048" layer="1"/>
@@
 <wire x1="5.0038" y1="50.165" x2="3.2025" y2="50.165" width="0.3048" layer="1"/>
 <wire x1="3.2025" y1="50.165" x2="2.8125" y2="49.775" width="0.3048" layer="1"/>
+<contactref element="IC9" pad="5"/>
+<wire x1="55.9625" y1="24.4625" x2="56.5" y2="25" width="0.3048" layer="1"/>
+<wire x1="56.5" y1="25" x2="56.875" y2="25" width="0.3048" layer="1"/>
+<via x="56.875" y="25" extent="1-16" drill="0.6" shape="octagon"/>
+<wire x1="56.875" y1="25" x2="57.1875" y2="25" width="0.3048" layer="16"/>
 </signal>
 <signal name="NRST">
